File: gw-glitchbus-proto2.sch (KiCad schematic (older format))
At the start: 7 parts, among them J1 GLITCHBUS, J2 GLITCHBUS

Commit message: Updating schematic for *BSELECTED, new library paths
Parts:
- J1, J2: symbol computer_busses:GLITCHBUS -> gw_computer_busses:GLITCHBUS_1.0
Connections:
- net GND: no longer J1.29 (GND), J2.29 (GND)
- new net *BSELECTED: J1.29 (*BSELECTED), J2.29 (*BSELECTED)
Other:
- moved on the sheet: C1, W1, W2, W3, W4
