File: gw-glitchbus-proto2.kicad_pcb (KiCad board)
At the start: 2 copper layers, 129.5 x 104.1 mm, 1636 parts, among them J1 GLITCHBUS, J2 GLITCHBUS

Commit message: Updating schematic for *BSELECTED, new library paths
Connections:
- J1 pad 29: GND -> *BSELECTED
- J2 pad 29: GND -> *BSELECTED
Routing:
- net *BSELECTED: track 0.00 -> 15.0 mm
Other:
- board text added: "*BSEL"
Changed lines of the file:
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@@
-(kicad_pcb (version 20171130) (host pcbnew 5.1.2)
+(kicad_pcb (version 20171130) (host pcbnew "(5.0.1-3-g963ef8bb5)")
   (general
     (thickness 1.6)
-    (drawings 78)
-    (tracks 138)
+    (drawings 80)
+    (tracks 142)
     (zones 0)
     (modules 1636)
-    (nets 35)
+    (nets 36)
   )
   (page USLetter)
@@
     (zone_45_only yes)
     (trace_min 0.2)
+    (segment_width 0.254)
+    (edge_width 0.254)
     (via_size 0.8128)
     (via_drill 0.4064)
@@
     (uvia_min_size 0)
     (uvia_min_drill 0)
-    (edge_width 0.254)
-    (segment_width 0.254)
     (pcb_text_width 0.254)
     (pcb_text_size 1.27 1.27)
@@
     (pad_drill 3.048)
     (pad_to_mask_clearance 0.2)
+    (solder_mask_min_width 0.25)
     (aux_axis_origin 0 0)
     (visible_elements FFFFFF7F)
@@
   (net 33 BD6)
   (net 34 BD7)
+  (net 35 *BSELECTED)
   (net_class Default "This is the default net class."
     (clearance 0.2)
@@
     (add_net *BMASK)
     (add_net *BRESET)
+    (add_net *BSELECTED)
     (add_net *BSTART)
     (add_net BA0)
@@
       (net 25 *BINT))
     (pad 29 thru_hole oval (at 0 35.56 90) (size 1.7272 1.7272) (drill 1.016) (layers *.Cu *.Mask)
-      (net 2 GND))
+      (net 35 *BSELECTED))
     (pad 30 thru_hole oval (at 2.54 35.56 90) (size 1.7272 1.7272) (drill 1.016) (layers *.Cu *.Mask)
       (net 26 BREADY))
@@
       (net 26 BREADY))
     (pad 29 thru_hole oval (at 0 35.56 90) (size 1.7272 1.7272) (drill 1.016) (layers *.Cu *.Mask)
-      (net 2 GND))
+      (net 35 *BSELECTED))
     (pad 28 thru_hole oval (at 2.54 33.02 90) (size 1.7272 1.7272) (drill 1.016) (layers *.Cu *.Mask)
       (net 25 *BINT))
@@
     )
   )
+  (gr_text *BSEL (at 175.26 140.335 270) (layer F.SilkS)
+    (effects (font (size 1.27 1.27) (thickness 0.254)) (justify left))
+  )
+  (gr_text *BSEL (at 175.26 140.335 270) (layer B.Mask)
+    (effects (font (size 1.27 1.27) (thickness 0.254)) (justify right mirror))
+  )
   (gr_line (start 69.85 52.07) (end 71.12 52.07) (layer Edge.Cuts) (width 0.254))
   (gr_line (start 69.85 53.34) (end 69.85 52.07) (layer Edge.Cuts) (width 0.254))
@@
   (segment (start 186.69 139.7) (end 186.69 137.16) (width 0.3048) (layer F.Cu) (net 34))
   (segment (start 186.69 137.16) (end 185.42 135.89) (width 0.3048) (layer F.Cu) (net 34))
+  (segment (start 175.26 152.4) (end 173.99 151.13) (width 0.3048) (layer F.Cu) (net 35))
+  (segment (start 173.99 151.13) (end 173.99 140.97) (width 0.3048) (layer F.Cu) (net 35))
+  (segment (start 173.99 140.97) (end 175.26 139.7) (width 0.3048) (layer F.Cu) (net 35))
+  (segment (start 175.26 139.7) (end 175.26 138.43) (width 0.3048) (layer F.Cu) (net 35))
   (zone (net 2) (net_name GND) (layer B.Cu) (hatch edge 0.508)
     (connect_pads (clearance 0.381))

Commit message: Updating to KiCAD 8
Other:
- net class Default removed
